File: macro_pad/macro_pad.sch (KiCad schematic (older format))
At the start: 51 parts, among them K01 KEYSW

Commit message: Everything but the OLED added
Parts:
- removed U?: IS31FL3731-QF, Package_DFN_QFN:QFN-28-1EP_4x4mm_P0.4mm_EP2.3x2.3mm, symbol Driver_LED:IS31FL3731-QF
- added D? (x14): LED, symbol Device:LED
- added LDO6AJSA?: LDO6AJSA, symbol Driver_LED:LDO6AJSA
- added U?: 74HC237, symbol 74xx:74HC237
- K01, K? (x17): symbol TMK_Keyboard_Parts:KEYSW -> macro_pad-rescue:KEYSW-TMK_Keyboard_Parts
- U?: symbol MCU_Pro_Micro:ProMicro -> macro_pad-rescue:ProMicro-MCU_Pro_Micro
Connections:
- net at U?.1 (TX): now also K01.1, K?.1, K?.1, K?.1, K?.1, SW?.S2
- net at U?.10 (E6): now also U?.1 (A0)
- net at U?.12 (B5): now also LDO6AJSA?.2 (CE)
- net at U?.13 (B6): now also SW?.B, SW?.B
- net at U?.14 (B2): now also SW?.A, U?.15 (B3)
- net at U?.16 (B1): now also SW?.A
- net at U?.17 (F7): now also SW?.B
- net at U?.18 (F6): now also SW?.A
- net at U?.19 (F5): now also SW?.B
- net at U?.2 (RX): now also K?.1, K?.1, K?.1, K?.1, K?.1, SW?.S2
- net at U?.20 (F4): now also SW?.A
- net at U?.21 (VCC): now also LDO6AJSA?.1 (V1), U?.16 (VCC)
- net at U?.3 (GND): now also K?.1, K?.1, K?.1, K?.1, K?.1, SW?.S2
- net at U?.4 (GND): now also SW?.C, SW?.C, SW?.C, SW?.C, LDO6AJSA?.3 (GND), U?.8 (GND)
- net at U?.7 (D4): now also K?.1, K?.1, K?.1, SW?.S2
- net at U?.8 (C6): now also U?.3 (A2)
- net at U?.9 (D7): now also U?.2 (A1)
- net at K01.2: now also D?.1 (K); no longer D?.2 (A)
- net at K?.2: now also D?.1 (K); no longer D?.2 (A) (x17)
- net at SW?.S1: now also D?.1 (K); no longer D?.2 (A) (x4)
- net at D?.1 (K): now also D?.1 (K), D?.1 (K), D?.1 (K), D?.1 (K), D?.1 (K), D?.1 (K), D?.1 (K), D?.1 (K), D?.1 (K), D?.1 (K), D?.1 (K), D?.1 (K), D?.1 (K), D?.1 (K), D?.1 (K), D?.1 (K), D?.1 (K)
- net at D?.2 (A): now also D?.2 (A), D?.2 (A), D?.2 (A), D?.2 (A), D?.2 (A), D?.2 (A), D?.2 (A), D?.2 (A), D?.2 (A), D?.2 (A), D?.2 (A), D?.2 (A), D?.2 (A), D?.2 (A), D?.2 (A), D?.2 (A), D?.2 (A), LDO6AJSA?.4 (LED)
- new net: D?.2 (A), D?.2 (A), D?.2 (A), D?.2 (A), U?.10 (Y5)
- new net: D?.2 (A), D?.2 (A), D?.2 (A), U?.11 (Y4)
- new net: D?.2 (A), D?.2 (A), D?.2 (A), D?.2 (A), U?.12 (Y3)
- new net: D?.2 (A), D?.2 (A), D?.2 (A), U?.13 (Y2)
- new net: D?.2 (A), D?.2 (A), D?.2 (A), D?.2 (A), U?.14 (Y1)
- new net: D?.2 (A), D?.2 (A), D?.2 (A), D?.2 (A), U?.15 (Y0)
Other:
- moved on the sheet: D?, K01, K?, SW?, U?
